File: proyecto_1/RERLAY_GROUP.kicad_sch (KiCad schematic)
At the start: 10 parts, among them U1 ULN2003A, U2 AZ921

Commit message: nuevos circuitos de pcb
Parts:
- added D5: LED, symbol Device:LED
- added R5: 1k, symbol Device:R
- added U3, U4, U5, U6: AZ921, symbol nuevo simbolos:AZ921
Connections:
- net +12V: now also R5.2
- net CON-FAN-C: now also U4.3, U5.3, U6.3
- net CON-FAN1: now also U4.4
- net CON-FAN2: now also U5.4
- net CON-FAN3: now also U6.4
- net CON-OUT1A: now also U2.4
- net CON-OUT1B: now also U2.3
- net CON-OUT2A: now also U3.4
- net CON-OUT2B: now also U3.3
- net VCC: now reaches U2.1
- net VCC: now also U3.1, U4.1, U5.1
- net at U2.2: now also D1.1 (K), U1.16 (O1)
- net at U1.12 (O5): now also D5.1 (K)
- net at D3.1 (K), U1.14 (O3): now also U4.2
- net at D2.1 (K), U1.15 (O2): now also U3.2
- net at D4.2 (A), R4.1: now also U5.2
- new net: D5.2 (A), R5.1, U6.1
Other:
- moved on the sheet: U2
