File: proyecto_1/CONTROL.kicad_sch (KiCad schematic)
At the start: 0 parts

Commit message: se completo el micro
Parts:
- added C5, C7: 0.1, symbol Device:C
- added C6: 22, symbol Device:C
- added D12: LED, symbol Device:LED
- added J7: Screw_Terminal_01x06, Connector_PinHeader_2.54mm:PinHeader_2x03_P2.54mm_Vertical, symbol Connector:Screw_Terminal_01x06
- added J8: Conn_ARM_JTAG_SWD_10, Connector_PinHeader_2.54mm:PinHeader_2x05_P2.54mm_Vertical, symbol Connector:Conn_ARM_JTAG_SWD_10
- added R26: 22k, symbol Device:R
- added R27: R, symbol Device:R
- added U13: ESP32-WROOM-32, RF_Module:ESP32-WROOM-32, symbol RF_Module:ESP32-WROOM-32
Connections:
- net COM_RS485_LCD: now also U13.6 (IO34)
- net CON_RS485_EXT: now also U13.7 (IO35)
- net INPUT_1_MICRO: now also U13.25 (IO0)
- net INPUT_2_MICRO: now also U13.29 (IO5)
- net INPUT_3_MICRO: now also U13.24 (IO2)
- net INPUT_4_MICRO: now also U13.26 (IO4)
- net RLY_FAN1_MICRO: now also U13.10 (IO25)
- net RLY_FAN2_MICRO: now also U13.11 (IO26)
- net RLY_FAN3_MICRO: now also U13.12 (IO27)
- net RLY_OUT1_MICRO: now also U13.36 (IO22)
- net RLY_OUT2_MICRO: now also U13.37 (IO23)
- net Rx_RS485_EXT: now also U13.27 (IO16)
- net Rx_RS485_LCD: now also U13.34 (RXD0/IO3)
- net Tx_RS485_EXT: now also U13.28 (IO17)
- net Tx_RS485_LCD: now also U13.35 (TXD0/IO1)
- new net: J7.2 (Pin_2), U13.30 (IO18)
- new net: J7.3 (Pin_3), U13.8 (IO32)
- new net: J7.4 (Pin_4), U13.31 (IO19)
- new net: J7.6 (Pin_6), U13.33 (IO21)
- new net: D12.2 (A), R27.1
- new net: C5.2, R26.2, U13.3 (EN)
- new net: J8.2 (SWDIO/TMS), U13.13 (IO14)
- new net: J8.8 (NC/TDI), U13.14 (IO12)
- new net: J8.4 (SWDCLK/TCK), U13.16 (IO13)
- new net: J8.6 (SWO/TDO), U13.23 (IO15)
- new net: D12.1 (K), U13.9 (IO33)
- new net GND: C6.2, C7.2, J7.5 (Pin_5), J8.3 (GND), J8.5 (GND), U13.1 (GND), U13.15 (GND), U13.38 (GND), U13.39 (GND)
- new net VCC: J8.1 (VTref)
- new net VDD: C5.1, C6.1, C7.1, J7.1 (Pin_1), J8.10 (~{RESET}), R26.1, R27.2, U13.2 (VDD)
- no-connect marks 0 -> 1
