File: proyecto_1/RS-485-LCD.kicad_sch (KiCad schematic)
At the start: 0 parts

Commit message: agregados al esquematico
Parts:
- added R28: R, symbol Device:R
- added U16: SP485ECN-L, SOIC127P600X175-8N, symbol SP485ECN-L:SP485ECN-L
- added U17: SMBJ12CA, nuevo simbolo:SMBJ12CA, symbol nuevo simbolos:SMBJ12CA
Connections:
- net COM_RS485_LCD: now also R28.1
- net Rx_RS485_LCD: now also U16.4 (DI)
- net Tx_RS485_LCD: now also U16.1 (RO)
- new net VCC: U16.8 (VCC)
Changed lines of the file:
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@@
 (kicad_sch (version 20230121) (generator eeschema)
   (paper "A4")
-  (hierarchical_label "Tx_RS485_LCD" (shape bidirectional) (at 74.93 57.15 0) (fields_autoplaced)
+  (junction (at 94.742 94.5896) (diameter 0) (color 0 0 0 0)
+  )
+  (wire (pts (xy 94.742 92.1004) (xy 94.742 94.5896))
+    (stroke (width 0) (type default))
+  )
+  (wire (pts (xy 84.328 94.5896) (xy 83.0072 94.5896))
+    (stroke (width 0) (type default))
+  )
+  (wire (pts (xy 97.0788 84.4296) (xy 97.0788 84.4804))
+    (stroke (width 0) (type default))
+  )
+  (wire (pts (xy 97.0788 94.6404) (xy 94.742 94.6404))
+    (stroke (width 0) (type default))
+  )
+  (wire (pts (xy 96.8756 83.7184) (xy 96.8756 84.4296))
+    (stroke (width 0) (type default))
+  )
+  (wire (pts (xy 94.742 94.5896) (xy 94.742 94.6404))
+    (stroke (width 0) (type default))
+  )
+  (wire (pts (xy 92.0496 94.5896) (xy 94.742 94.5896))
+    (stroke (width 0) (type default))
+  )
+  (wire (pts (xy 97.1296 83.7184) (xy 96.8756 83.7184))
+    (stroke (width 0) (type default))
+  )
+  (wire (pts (xy 90.5256 88.646) (xy 90.5256 89.5604))
+    (stroke (width 0) (type default))
+  )
+  (wire (pts (xy 96.8756 84.4296) (xy 97.0788 84.4296))
+    (stroke (width 0) (type default))
+  )
+  (wire (pts (xy 90.4748 88.646) (xy 90.5256 88.646))
+    (stroke (width 0) (type default))
+  )
+  (wire (pts (xy 90.5256 89.5604) (xy 97.0788 89.5604))
+    (stroke (width 0) (type default))
+  )
+  (wire (pts (xy 97.1296 80.6704) (xy 97.1296 83.7184))
+    (stroke (width 0) (type default))
+  )
+  (wire (pts (xy 132.6388 89.5604) (xy 138.7856 89.5604))
+    (stroke (width 0) (type default))
+  )
+  (wire (pts (xy 94.742 92.1004) (xy 97.1296 92.1004))
+    (stroke (width 0) (type default))
+  )
+  (hierarchical_label "Tx_RS485_LCD" (shape bidirectional) (at 138.7348 89.5604 0) (fields_autoplaced)
     (effects (font (size 1.27 1.27)) (justify left))
   )
-  (hierarchical_label "COM_RS485_LCD" (shape bidirectional) (at 74.93 64.77 0) (fields_autoplaced)
-    (effects (font (size 1.27 1.27)) (justify left))
+  (hierarchical_label "COM_RS485_LCD" (shape bidirectional) (at 83.058 94.5896 180) (fields_autoplaced)
+    (effects (font (size 1.27 1.27)) (justify right))
   )
   (hierarchical_label "CON-LCDA-" (shape bidirectional) (at 74.93 45.72 0) (fields_autoplaced)
@@
     (effects (font (size 1.27 1.27)) (justify left))
   )
-  (hierarchical_label "Rx_RS485_LCD" (shape bidirectional) (at 74.93 60.96 0) (fields_autoplaced)
-    (effects (font (size 1.27 1.27)) (justify left))
+  (hierarchical_label "Rx_RS485_LCD" (shape bidirectional) (at 90.4748 88.646 180) (fields_autoplaced)
+    (effects (font (size 1.27 1.27)) (justify right))
+  )
+  (symbol (lib_id "nuevo simbolos:SMBJ12CA") (at 154.8892 77.8256 0) (unit 1)
+    (in_bom yes) (on_board yes) (dnp no) (fields_autoplaced)
+    (property "Reference" "U17" (at 157.48 70.7136 0)
+      (effects (font (size 1.27 1.27)) (justify left))
+    )
+    (property "Value" "SMBJ12CA" (at 157.48 73.2536 0)
+      (effects (font (size 1.27 1.27)) (justify left))
+    )
+    (property "Footprint" "nuevo simbolo:SMBJ12CA" (at 161.7472 72.2376 0)
+      (effects (font (size 1.27 1.27)) hide)
+    )
+    (property "Datasheet" "https://pdf1.alldatasheet.com/datasheet-pdf/view/568474/SOCAY/SMBJ12CA.html" (at 161.7472 72.2376 0)
+      (effects (font (size 1.27 1.27)) hide)
+    )
+    (pin "1")
+    (pin "2")
+    (instances
+      (project "proyecto_1"
+        (path "/a26e3056-8779-457a-a9c5-797bfba96834/0a54ac0f-412f-4dea-a78e-7d38c349c597/a0c76e55-fe1e-4057-89cd-2a04e6220d2e"
+          (reference "U17") (unit 1)
+        )
+      )
+    )
+  )
+  (symbol (lib_id "power:VCC") (at 97.1296 80.6704 0) (unit 1)
+    (in_bom yes) (on_board yes) (dnp no) (fields_autoplaced)
+    (property "Reference" "#PWR042" (at 97.1296 84.4804 0)
+      (effects (font (size 1.27 1.27)) hide)
+    )
+    (property "Value" "VCC" (at 97.1296 77.47 0)
+      (effects (font (size 1.27 1.27)))
+    )
+    (property "Footprint" "" (at 97.1296 80.6704 0)
+      (effects (font (size 1.27 1.27)) hide)
+    )
+    (property "Datasheet" "" (at 97.1296 80.6704 0)
+      (effects (font (size 1.27 1.27)) hide)
+    )
+    (pin "1")
+    (instances
+      (project "proyecto_1"
+        (path "/a26e3056-8779-457a-a9c5-797bfba96834/0a54ac0f-412f-4dea-a78e-7d38c349c597/a0c76e55-fe1e-4057-89cd-2a04e6220d2e"
+          (reference "#PWR042") (unit 1)
+        )
+      )
+    )
+  )
+  (symbol (lib_id "SP485ECN-L:SP485ECN-L") (at 97.0788 84.4804 0) (unit 1)
+    (in_bom yes) (on_board yes) (dnp no) (fields_autoplaced)
+    (property "Reference" "U16" (at 114.8588 74.93 0)
+      (effects (font (size 1.27 1.27)))
+    )
+    (property "Value" "SP485ECN-L" (at 114.8588 77.47 0)
+      (effects (font (size 1.27 1.27)))
+    )
+    (property "Footprint" "SOIC127P600X175-8N" (at 97.0788 84.4804 0)
+      (effects (font (size 1.27 1.27)) (justify bottom) hide)
+    )
+    (property "Datasheet" "" (at 97.0788 84.4804 0)
+      (effects (font (size 1.27 1.27)) hide)
+    )
+    (property "SUPPLIER" "Sipex Corporation" (at 97.0788 84.4804 0)
+      (effects (font (size 1.27 1.27)) (justify bottom) hide)
+    )
+    (property "OC_FARNELL" "1831933" (at 97.0788 84.4804 0)
+      (effects (font (size 1.27 1.27)) (justify bottom) hide)
+    )
+    (property "OC_NEWARK" "24R0570" (at 97.0788 84.4804 0)
+      (effects (font (size 1.27 1.27)) (justify bottom) hide)
+    )
+    (property "MPN" "SP485ECN-L" (at 97.0788 84.4804 0)
+      (effects (font (size 1.27 1.27)) (justify bottom) hide)
+    )
+    (property "PACKAGE" "SOIC-8" (at 97.0788 84.4804 0)
+      (effects (font (size 1.27 1.27)) (justify bottom) hide)
+    )
+    (pin "1")
+    (pin "2")
+    (pin "3")
+    (pin "4")
+    (pin "5")
+    (pin "6")
+    (pin "7")
+    (pin "8")
+    (instances
+      (project "proyecto_1"
+        (path "/a26e3056-8779-457a-a9c5-797bfba96834/0a54ac0f-412f-4dea-a78e-7d38c349c597/a0c76e55-fe1e-4057-89cd-2a04e6220d2e"
+          (reference "U16") (unit 1)
+        )
+      )
+    )
+  )
+  (symbol (lib_id "Device:R") (at 88.138 94.5896 90) (unit 1)
+    (in_bom yes) (on_board yes) (dnp no) (fields_autoplaced)
+    (property "Reference" "R28" (at 88.138 90.17 90)
+      (effects (font (size 1.27 1.27)))
+    )
+    (property "Value" "R" (at 88.138 92.71 90)
+      (effects (font (size 1.27 1.27)))
+    )
+    (property "Footprint" "" (at 88.138 96.3676 90)
+      (effects (font (size 1.27 1.27)) hide)
+    )
+    (property "Datasheet" "~" (at 88.138 94.5896 0)
+      (effects (font (size 1.27 1.27)) hide)
+    )
+    (pin "1")
+    (pin "2")
+    (instances
+      (project "proyecto_1"
+        (path "/a26e3056-8779-457a-a9c5-797bfba96834/0a54ac0f-412f-4dea-a78e-7d38c349c597/a0c76e55-fe1e-4057-89cd-2a04e6220d2e"
+          (reference "R28") (unit 1)
+        )
+      )
+    )
   )
 )

Commit message: avance del proyecto
Parts:
- added C8, C9: C, symbol Device:C
- added D13: SM712_SOT23, Package_TO_SOT_SMD:SOT-23, symbol Diode:SM712_SOT23
- added R29, R30: R, symbol Device:R
Connections:
- net CON-LCDA-: now also R30.2
- net CON-LCDB+: now also R29.2
- net VCC: now also C8.1, C9.1
- net at U17.2: now also U16.6 (A), D13.2 (A2), R29.1
- net at U16.2 (~RE): now also R28.2, U16.3 (DE)
- net GND: now reaches U16.5 (GND)
- net GND: now also C8.2, C9.2, D13.3 (common)
- net at U16.7 (B): now also R30.1
Other:
- moved on the sheet: U17
