File: proyecto_1/POWER_SUPPLY.kicad_sch (KiCad schematic)
At the start: 0 parts

Commit message: agregados al esquematico
Parts:
- added U14: B0505S-W2R2, nuevo simbolo:B0505S-W2R2, symbol nuevo simbolos:B0505S-W2R2
- added U15: fuse_CC12H1.5A-TR, nuevo simbolo:CC12H1.5A-TR, symbol nuevo simbolos:fuse_CC12H1.5A-TR
Changed lines of the file:
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@@
     (effects (font (size 1.27 1.27)) (justify left))
   )
+  (symbol (lib_id "nuevo simbolos:fuse_CC12H1.5A-TR") (at 55.88 111.76 0) (unit 1)
+    (in_bom yes) (on_board yes) (dnp no) (fields_autoplaced)
+    (property "Reference" "U15" (at 55.753 106.68 0)
+      (effects (font (size 1.27 1.27)))
+    )
+    (property "Value" "fuse_CC12H1.5A-TR" (at 55.753 109.22 0)
+      (effects (font (size 1.27 1.27)))
+    )
+    (property "Footprint" "nuevo simbolo:CC12H1.5A-TR" (at 55.88 109.22 0)
+      (effects (font (size 1.27 1.27)) hide)
+    )
+    (property "Datasheet" "https://www.mouser.com/datasheet/2/87/eaton_cc12h_high_i2t_chip_fuses_data_sheet-1608530.pdf" (at 55.88 107.442 0)
+      (effects (font (size 1.27 1.27)) hide)
+    )
+    (pin "1")
+    (pin "2")
+    (instances
+      (project "proyecto_1"
+        (path "/a26e3056-8779-457a-a9c5-797bfba96834/0a54ac0f-412f-4dea-a78e-7d38c349c597/9d91a05e-a16e-4a79-b8a8-d7453eb27381"
+          (reference "U15") (unit 1)
+        )
+      )
+    )
+  )
+  (symbol (lib_id "nuevo simbolos:B0505S-W2R2") (at 167.64 83.82 0) (unit 1)
+    (in_bom yes) (on_board yes) (dnp no) (fields_autoplaced)
+    (property "Reference" "U14" (at 167.513 76.2 0)
+      (effects (font (size 1.27 1.27)))
+    )
+    (property "Value" "B0505S-W2R2" (at 167.513 78.74 0)
+      (effects (font (size 1.27 1.27)))
+    )
+    (property "Footprint" "nuevo simbolo:B0505S-W2R2" (at 169.672 88.646 0)
+      (effects (font (size 1.27 1.27)) hide)
+    )
+    (property "Datasheet" "https://www.mouser.com/datasheet/2/942/SF_IB-1508439.pdf" (at 169.926 90.424 0)
+      (effects (font (size 1.27 1.27)) hide)
+    )
+    (pin "1")
+    (pin "2")
+    (pin "3")
+    (pin "4")
+    (instances
+      (project "proyecto_1"
+        (path "/a26e3056-8779-457a-a9c5-797bfba96834/0a54ac0f-412f-4dea-a78e-7d38c349c597/9d91a05e-a16e-4a79-b8a8-d7453eb27381"
+          (reference "U14") (unit 1)
+        )
+      )
+    )
+  )
 )

Commit message: avance del proyecto
Parts:
- added C10: C, symbol Device:C
- added D13: SM712_SOT23, Package_TO_SOT_SMD:SOT-23, symbol Diode:SM712_SOT23
- added D14: 1SMA5918BT3G, Diode_SMD:D_SMB, symbol nuevo simbolos:1SMA5918BT3G
- added PS1: HLK-PM12, Converter_ACDC:Converter_ACDC_HiLink_HLK-PMxx, symbol Converter_ACDC:HLK-PM12
- added V1: MOV-10D561K, MOV-10D561, symbol MOV-10D561K:MOV-10D561K
Changed lines of the file:
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@@
+    )
+  )
+  (symbol (lib_id "Converter_ACDC:HLK-PM12") (at 112.4204 106.8832 0) (unit 1)
+    (in_bom yes) (on_board yes) (dnp no) (fields_autoplaced)
+    (property "Reference" "PS1" (at 112.4204 99.06 0)
+      (effects (font (size 1.27 1.27)))
+    )
+    (property "Value" "HLK-PM12" (at 112.4204 101.6 0)
+      (effects (font (size 1.27 1.27)))
+    )
+    (property "Footprint" "Converter_ACDC:Converter_ACDC_HiLink_HLK-PMxx" (at 112.4204 114.5032 0)
+      (effects (font (size 1.27 1.27)) hide)
+    )
+    (property "Datasheet" "http://www.hlktech.net/product_detail.php?ProId=56" (at 122.5804 115.7732 0)
+      (effects (font (size 1.27 1.27)) hide)
+    )
+    (pin "1")
+    (pin "2")
+    (pin "3")
+    (pin "4")
+    (instances
+      (project "proyecto_1"
+        (path "/a26e3056-8779-457a-a9c5-797bfba96834/0a54ac0f-412f-4dea-a78e-7d38c349c597/9d91a05e-a16e-4a79-b8a8-d7453eb27381"
+          (reference "PS1") (unit 1)
+        )
+      )
+    )
+  )
+  (symbol (lib_id "Diode:SM712_SOT23") (at 136.8044 95.6056 0) (unit 1)
+    (in_bom yes) (on_board yes) (dnp no) (fields_autoplaced)
+    (property "Reference" "D13" (at 136.8044 90.2716 0)
+      (effects (font (size 1.27 1.27)))
+    )
+    (property "Value" "SM712_SOT23" (at 136.8044 92.8116 0)
+      (effects (font (size 1.27 1.27)))
+    )
+    (property "Footprint" "Package_TO_SOT_SMD:SOT-23" (at 136.8044 104.4956 0)
+      (effects (font (size 1.27 1.27)) hide)
+    )
+    (property "Datasheet" "https://www.littelfuse.com/~/media/electronics/datasheets/tvs_diode_arrays/littelfuse_tvs_diode_array_sm712_datasheet.pdf.pdf" (at 132.9944 95.6056 0)
+      (effects (font (size 1.27 1.27)) hide)
+    )
+    (pin "1")
+    (pin "2")
+    (pin "3")
+    (instances
+      (project "proyecto_1"
+        (path "/a26e3056-8779-457a-a9c5-797bfba96834/0a54ac0f-412f-4dea-a78e-7d38c349c597/a0c76e55-fe1e-4057-89cd-2a04e6220d2e"
+          (reference "D13") (unit 1)
+        )
+        (path "/a26e3056-8779-457a-a9c5-797bfba96834/0a54ac0f-412f-4dea-a78e-7d38c349c597/9d91a05e-a16e-4a79-b8a8-d7453eb27381"
+          (reference "D15") (unit 1)
+        )
+      )
+    )
+  )
+  (symbol (lib_id "Device:C") (at 68.7832 84.7852 0) (unit 1)
+    (in_bom yes) (on_board yes) (dnp no) (fields_autoplaced)
+    (property "Reference" "C10" (at 72.39 84.1502 0)
+      (effects (font (size 1.27 1.27)) (justify left))
+    )
+    (property "Value" "C" (at 72.39 86.6902 0)
+      (effects (font (size 1.27 1.27)) (justify left))
+    )
+    (property "Footprint" "" (at 69.7484 88.5952 0)
+      (effects (font (size 1.27 1.27)) hide)
+    )
+    (property "Datasheet" "~" (at 68.7832 84.7852 0)
+      (effects (font (size 1.27 1.27)) hide)
+    )
+    (pin "1")
+    (pin "2")
+    (instances
+      (project "proyecto_1"
+        (path "/a26e3056-8779-457a-a9c5-797bfba96834/0a54ac0f-412f-4dea-a78e-7d38c349c597/9d91a05e-a16e-4a79-b8a8-d7453eb27381"
+          (reference "C10") (unit 1)
+        )
+      )
     )
   )
@@
         )
       )
+    )
+  )
+  (symbol (lib_id "MOV-10D561K:MOV-10D561K") (at 77.6732 119.0752 0) (unit 1)
+    (in_bom yes) (on_board yes) (dnp no) (fields_autoplaced)
+    (property "Reference" "V1" (at 77.6732 113.03 0)
+      (effects (font (size 1.27 1.27)))
+    )
+    (property "Value" "MOV-10D561K" (at 77.6732 115.57 0)
+      (effects (font (size 1.27 1.27)))
+    )
+    (property "Footprint" "MOV-10D561" (at 77.6732 119.0752 0)
+      (effects (font (size 1.27 1.27)) (justify bottom) hide)
+    )
+    (property "Datasheet" "" (at 77.6732 119.0752 0)
+      (effects (font (size 1.27 1.27)) hide)
+    )
+    (pin "1")
+    (pin "2")
+    (instances
+      (project "proyecto_1"
+        (path "/a26e3056-8779-457a-a9c5-797bfba96834/0a54ac0f-412f-4dea-a78e-7d38c349c597/9d91a05e-a16e-4a79-b8a8-d7453eb27381"
+          (reference "V1") (unit 1)
+        )
+      )
+    )
+  )
+  (symbol (lib_id "nuevo simbolos:1SMA5918BT3G") (at 95.4024 71.9328 0) (unit 1)
+    (in_bom yes) (on_board yes) (dnp no) (fields_autoplaced)
+    (property "Reference" "D14" (at 95.2119 66.04 0)
+      (effects (font (size 1.27 1.27)))
+    )
+    (property "Value" "1SMA5918BT3G" (at 95.2119 68.58 0)
+      (effects (font (size 1.27 1.27)))
+    )
+    (property "Footprint" "Diode_SMD:D_SMB" (at 95.4024 78.2828 0)
+      (effects (font (size 1.27 1.27)) hide)
+    )
+    (property "Datasheet" "https://www.mouser.com/datasheet/2/308/1SMA5913BT3_D-2309368.pdf" (at 94.3864 80.5688 0)
+      (effects (font (size 1.27 1.27)) hide)
+    )
+    (pin "1")
+    (pin "2")
+    (instances
+      (project "proyecto_1"
+        (path "/a26e3056-8779-457a-a9c5-797bfba96834/0a54ac0f-412f-4dea-a78e-7d38c349c597/9d91a05e-a16e-4a79-b8a8-d7453eb27381"
+          (reference "D14") (unit 1)
+        )
+      )

Commit message: fuente
Parts:
- added D16: LED, symbol Device:LED
- added D17: 1SMA5918BT3G, Diode_SMD:D_SMB, symbol nuevo simbolos:1SMA5918BT3G
- added R31: R, symbol Device:R
- added U18, U19: fuse_CC12H1.5A-TR, nuevo simbolo:CC12H1.5A-TR, symbol nuevo simbolos:fuse_CC12H1.5A-TR
Connections:
- net CON-DC+: now also U15.2, R31.1
- net CON-DC-: now also D16.1 (K), U18.2
- net CON-L1: now also U19.1
- net CON-NEUT: now also PS1.1 (AC/L), V1.1
- net VCC: now reaches U15.1
- net VCC: now also C10.1, D13.1 (A1), PS1.4 (+Vout)
- net at PS1.2 (AC/N): now also V1.2, U19.2
- net GND: now reaches PS1.3 (-Vout)
- net GND: now also C10.2, U18.1
- new net: D16.2 (A), R31.2
Other:
- moved on the sheet: C10, D13, D14, U14, U15, V1
